Commit message: colcon build and launch/urdf file fix

File: src/youbot_description/urdf/youbot.urdf (robot description, URDF)
Before this commit: robot youbot, 20 links, 19 joints
Links:
- link arm_link_0: geometry collision mesh filename=package://youbot_description/meshes/youbot_arm/arm0_convex.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; visual mesh filename=package://youbot_description/meshes/youbot_arm/arm0.dae
- link arm_link_1: geometry collision mesh filename=package://youbot_description/meshes/youbot_arm/arm_joint_1_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; visual mesh filename=package://youbot_description/meshes/youbot_arm/arm1.dae
- link arm_link_2: geometry collision mesh filename=package://youbot_description/meshes/youbot_arm/arm_joint_2_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; visual mesh filename=package://youbot_description/meshes/youbot_arm/arm2.dae
- link arm_link_3: geometry collision mesh filename=package://youbot_description/meshes/youbot_arm/arm_joint_3_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; visual mesh filename=package://youbot_description/meshes/youbot_arm/arm3.dae
- link arm_link_4: geometry collision mesh filename=package://youbot_description/meshes/youbot_arm/arm_joint_4_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; visual mesh filename=package://youbot_description/meshes/youbot_arm/arm4.dae
- link arm_link_5: geometry collision mesh filename=package://youbot_description/meshes/youbot_arm/arm_joint_5_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; visual mesh filename=package://youbot_description/meshes/youbot_arm/arm5.dae
- link base_laser_front_link: geometry collision mesh filename=package://youbot_description/meshes/sensors/hokuyo_convex.d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; visual mesh filename=package://youbot_description/meshes/sensors/hokuyo.dae
- link base_link: geometry collision mesh filename=package://youbot_description/meshes/youbot_base/base_convex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; visual mesh filename=package://youbot_description/meshes/youbot_base/base.dae
- link plate_link: geometry collision mesh filename=package://youbot_description/meshes/youbot_plate/plate_conv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; visual mesh filename=package://youbot_description/meshes/youbot_plate/plate.dae
- link wheel_link_bl: geometry collision cylinder length=0.05 radius=0.05; visual mesh filename=package://youbot_description/meshes/youbot_base/back-left_w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
- link wheel_link_br: geometry collision cylinder length=0.05 radius=0.05; visual mesh filename=package://youbot_description/meshes/youbot_base/back-right_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
- link wheel_link_fl: geometry collision cylinder length=0.05 radius=0.05; visual mesh filename=package://youbot_description/meshes/youbot_base/front-left_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
- link wheel_link_fr: geometry collision cylinder length=0.05 radius=0.05; visual mesh filename=package://youbot_description/meshes/youbot_base/front-right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
